File: kicad/esim/esim.kicad_pcb (KiCad board)
At the start: 2 copper layers, 100 x 100 mm, 28 parts, among them J1 GND + TXD RXD, SW1 Reset, U1 AT89x51xxP, U2 CY62256-70PC, U3 CY62256-70PC, U4-ADRLO1 74LS245, U5-ADRHI1 74LS245, U6-DATA1 74LS245, Y1 22.1184Mhz

Commit message: freshly routed
Parts:
- removed REF1, REF2: PinHeader_2x31_P2.54mm_Vertical, Connector_PinHeader_2.54mm:PinHeader_2x31_P2.54mm_Vertical
- removed REF3, REF4, REF5, REF6: PinHeader_2x38_P2.54mm_Vertical, Connector_PinHeader_2.54mm:PinHeader_2x38_P2.54mm_Vertical
- added R3: 10k, Resistor_THT:R_Axial_DIN0204_L3.6mm_D1.6mm_P7.62mm_Horizontal, F.Cu at (18.0, 66.8)
- Y1: footprint Crystal:Crystal_HC52-6mm_Vertical -> Crystal:Crystal_HC49-U_Vertical
- moved R1 22.5 mm to (93.0, 48.5), turned to 90 degrees
- moved C1 2.82 mm to (80.3, 17.0), turned to 0 degrees
Connections:
- C1 pad 1: RES\ -> +5V
- C1 pad 2: GND -> RES
- R1 pad 1: +5V -> GND
- R1 pad 2: RES\ -> RES
- SW1 pad 1: GND -> +5V
- SW1 pad 2: RES\ -> RES
- U1 pad 9: RES\ -> RES
- U6-DATA1 pad 1: RAMWE\ -> Net-(U6-DATA1-A->B)
- U6-DATA1 pad 19: RAMOE\ -> RAMCE\
Routing:
- net RAMWE\: track 113.8 -> 65.0 mm, vias 2 -> 1
- net RES: track 0.00 -> 46.9 mm
- net /A4: track 52.4 -> 98.9 mm, vias 1 -> 2
- net RES\: track 44.6 -> 0.00 mm
- net OE\: track 104.8 -> 60.7 mm, vias 0 -> 3
- net +5V: track 248.2 -> 291.6 mm
- net /A6: track 53.8 -> 94.2 mm, vias 1 -> 0
- net /A3: track 94.9 -> 56.0 mm, vias 2 -> 0
- net RAMCE\: track 57.8 -> 93.7 mm, vias 1 -> 0
- net /RA12: track 105.6 -> 70.8 mm, vias 0 -> 1
- net /A8: track 80.8 -> 115.6 mm, vias 1 -> 2
- net /RA10: track 39.7 -> 72.9 mm, vias 2 -> 5
- net /A5: track 55.4 -> 81.0 mm
- net RAMOE\: track 87.1 -> 64.7 mm
- net /A12: track 98.4 -> 76.5 mm, vias 0 -> 3
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- removed copper zone on B.Cu, net (none)
- removed copper zone on F.Cu, net (none)
- removed copper zone on B.Cu, net GND
- removed copper zone on F.Cu, net GND
