File: kicad/esim/esim.kicad_sch (KiCad schematic)
At the start: 22 parts, among them J1 GND + TXD RXD, SW1 Reset, U1 AT89x51xxP, U2 CY62256-70PC, U3 CY62256-70PC, U4-ADRLO1 74LS245, U5-ADRHI1 74LS245, U6-DATA1 74LS245, Y1 22.1184Mhz

Commit message: freshly routed
Parts:
- added R3: 10k, Resistor_THT:R_Axial_DIN0204_L3.6mm_D1.6mm_P7.62mm_Horizontal, symbol Device:R
- Y1: footprint Crystal:Crystal_HC52-6mm_Vertical -> Crystal:Crystal_HC49-U_Vertical
Connections:
- net +5V: now also C1.1, SW1.1, R3.1; no longer R1.1
- net GND: now also R1.1; no longer C1.2, SW1.1
- net RAMCE\: now also U6-DATA1.19 (CE)
- net RAMOE\: no longer U6-DATA1.19 (CE)
- net RAMWE\: no longer U6-DATA1.1 (A->B)
- net RES\ renamed RES
- net RES: now also C1.2; no longer C1.1
- new net: R3.2, U6-DATA1.1 (A->B)
Other:
- moved on the sheet: C1, R1, R2, SW1
